Commit message: 修改launch

File: src/arm/model/arm.urdf (robot description, URDF)
Before this commit: robot arm, 5 links, 4 joints
Links:
- link base_link: geometry collision mesh filename=package://arm/model/base_link.STL; visual mesh filename=package://arm/model/base_link.STL
- link link1: geometry collision mesh filename=package://arm/model/link1.STL; visual mesh filename=package://arm/model/link1.STL
- link link2: geometry collision mesh filename=package://arm/model/link2.STL; visual mesh filename=package://arm/model/link2.STL
- link link3: geometry collision mesh filename=package://arm/model/link3.STL; visual mesh filename=package://arm/model/link3.STL
- link link4: geometry collision mesh filename=package://arm/model/link4.STL; visual mesh filename=package://arm/model/link4.STL
